File: hardware/canary.kicad_pcb (KiCad board)
At the start: 0 parts

Commit message: fix(hardware): rebuild schematic, optimize PCB layout and pass ERC/DRC
- Fix schematic corruption with standard KiCad 10 symbols and power flags (0 ERC violations)
- Reorganize PCB layout into compact 44x40mm board with tight decoupling (<5.2mm)
- Route clean GND, 5V, 3.3V power rails and signals on F.Cu/B.Cu with zero violations (0 DRC violations)
- Add .gitignore for KiCad temporary files
Parts:
- added C1: 100nF, Capacitor_SMD:C_1206_3216Metric, F.Cu at (63.3, 91.0)
- added C2: 10uF, Capacitor_SMD:C_1206_3216Metric, F.Cu at (56.7, 91.0)
- added D1: LED, LED_SMD:LED_1206_3216Metric, F.Cu at (72.0, 110.0)
- added R1: 220, Resistor_SMD:R_1206_3216Metric, F.Cu at (72.0, 103.0)
- added R2: 10k, Resistor_SMD:R_1206_3216Metric, F.Cu at (48.0, 103.0)
- added SW1: RST, Button_Switch_SMD:SW_SPST_PTS810, F.Cu at (48.0, 110.0)
- added U1: AMS1117-3.3, Package_TO_SOT_SMD:SOT-223-3_TabPin2, F.Cu at (60.0, 96.0)
Routing:
- net GND: track 0.00 -> 62.2 mm, vias 0 -> 5
- net +5V: track 0.00 -> 55.5 mm
- net +3.3V: track 0.00 -> 24.1 mm
- net RST_BTN: track 0.00 -> 8.40 mm
- net LED_OUT: track 0.00 -> 7.00 mm
Other:
- board outline added: 44 x 40 mm
- copper layers 0 -> 2
