File: hardware/canary.kicad_sch (KiCad schematic)
At the start: 0 parts

Commit message: fix(hardware): rebuild schematic, optimize PCB layout and pass ERC/DRC
- Fix schematic corruption with standard KiCad 10 symbols and power flags (0 ERC violations)
- Reorganize PCB layout into compact 44x40mm board with tight decoupling (<5.2mm)
- Route clean GND, 5V, 3.3V power rails and signals on F.Cu/B.Cu with zero violations (0 DRC violations)
- Add .gitignore for KiCad temporary files
Parts:
- added C1: 100nF, Capacitor_SMD:C_1206_3216Metric, symbol Device:C
- added C2: 10uF, Capacitor_SMD:C_1206_3216Metric, symbol Device:C
- added D1: LED, LED_SMD:LED_1206_3216Metric, symbol Device:LED
- added R1: 220, Resistor_SMD:R_1206_3216Metric, symbol Device:R
- added R2: 10k, Resistor_SMD:R_1206_3216Metric, symbol Device:R
- added SW1: RST, Button_Switch_SMD:SW_SPST_PTS810, symbol Switch:SW_Push
- added U1: AMS1117-3.3, Package_TO_SOT_SMD:SOT-223-3_TabPin2, symbol Regulator_Linear:AMS1117-3.3
Connections:
- new net +3.3V: C2.1, R1.1, U1.2 (VO)
- new net +5V: C1.1, R2.1, U1.3 (VI)
- new net GND: C1.2, C2.2, D1.2 (A), SW1.2, U1.1 (GND)
- new net LED_OUT: D1.1 (K), R1.2
- new net RST_BTN: R2.2, SW1.1

Commit message: fix(release): set title block revision, align BOM footprints and add risk waiver
Other:
- company: (none) -> BoardReadyOps
- title: (none) -> Canary Board
Changed lines of the file:
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@@
 	(generator_version "10.0")
 	(paper "A4")
+	(title_block
+		(title "Canary Board")
+		(date "2026-09-01")
+		(rev "1.0.0")
+		(company "BoardReadyOps")
+	)
 	(wire
 		(pts
